File: dc_shield.kicad_sch (KiCad schematic)
At the start: 33 parts, among them J101 Vdrive, J102 Power, J103 Analog, J104 Digital/PWM, J105 Digital/PWM, J106 DC, J107 DC, Q101 SUD50P06-15, U101 VR10S12, U102 AT24C256C-SSHL-T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

Commit message: Add current sensing
Signed-off-by: Benedikt Spranger <b.spranger@linutronix.de>
Parts:
- added C115, C116: 1n, Capacitor_SMD:C_0603_1608Metric, symbol Device:C
- added C117, C118: 100n, Capacitor_SMD:C_0603_1608Metric, symbol Device:C
- added D104, D105: 1N4448W, Diode_SMD:D_SOD-123, symbol Diode:1N4448W
- added R104, R105: 10k, Resistor_SMD:R_0402_1005Metric, symbol Device:R
- added R106, R107: 2k, Resistor_SMD:R_0402_1005Metric, symbol Device:R
- added U105, U106: ACS712ELCTR-05B, Package_SO:SOIC-8_3.9x4.9mm_P1.27mm, symbol Sensor_Current:ACS712xLCTR-05B
- U102, U103, U104: assemble (none) -> y
Connections:
- net +5V: now also U105.8 (VCC), U106.8 (VCC)
- net A0: now also C118.1, D104.1 (K)
- net A1: now also C117.1, D105.1 (K)
- net GND: now also C115.2, C116.2, C117.2, C118.2, R104.2, R105.2, U105.5 (GND), U106.5 (GND)
- net Vdrive: now also U105.1 (IP+), U105.2 (IP+), U106.1 (IP+), U106.2 (IP+); no longer C107.1, C108.1, C109.1, C110.1, C111.1, C112.1, U103.4 (VS), U104.4 (VS)
- new net: D104.2 (A), R104.1, R106.2
- new net: R107.1, U106.7 (VIOUT)
- new net: D105.2 (A), R105.1, R107.2
- new net: C116.1, U106.6 (FILTER)
- new net: R106.1, U105.7 (VIOUT)
- new net: C115.1, U105.6 (FILTER)
- new net VdriveA: C107.1, C108.1, C109.1, U104.4 (VS), U106.3 (IP-), U106.4 (IP-)
- new net VdriveB: C110.1, C111.1, C112.1, U103.4 (VS), U105.3 (IP-), U105.4 (IP-)
- no-connect marks 14 -> 12
Other:
- moved on the sheet: C107, C108, C109, C110, C111, C112

Commit message: Replace 5A current sensor by 20A variant
Signed-off-by: Benedikt Spranger <b.spranger@linutronix.de>
Parts:
- removed U105, U106: ACS712ELCTR-05B, Package_SO:SOIC-8_3.9x4.9mm_P1.27mm, symbol Sensor_Current:ACS712xLCTR-05B
- added U105, U106: ACS712ELCTR-20A, Package_SO:SOIC-8_3.9x4.9mm_P1.27mm, symbol Sensor_Current:ACS712xLCTR-20A
Connections:
- net +5V: now also U105.8 (VCC), U106.8 (VCC)
- net GND: now also U105.5 (GND), U106.5 (GND)
- net Vdrive: now also U105.1 (IP+), U105.2 (IP+), U106.1 (IP+), U106.2 (IP+)
- net VdriveA: now also U106.3 (IP-), U106.4 (IP-)
- net VdriveB: now also U105.3 (IP-), U105.4 (IP-)
- net at R107.1: now also U106.7 (VIOUT)
- net at C116.1: now also U106.6 (FILTER)
- net at R106.1: now also U105.7 (VIOUT)
- net at C115.1: now also U105.6 (FILTER)

Commit message: Update JLCPCB parts
Signed-off-by: Benedikt Spranger <b.spranger@linutronix.de>
Parts:
- C101: LCSC# C108343 -> C15849; Manufacture FH (Guangdong Fenghua Advanced Tech) -> Samsung Electro-Mechanics; SupplLink https://jlcpcb.com/partdetail/109562-0603F105M500NT/C108343 -> https://jlcpcb.com/partdetail/16531-CL10A105KB8NNNC/C15849; mpn 0603F105M500NT -> CL10A105KB8NNNC
- C102, C108, C111, C113, C114: LCSC# C329928 -> C13585; Manufacture TDK -> Samsung Electro-Mechanics; SupplLink https://jlcpcb.com/partdetail/Tdk-C3216X5R1H106KT000N/C3299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 -> https://jlcpcb.com/partdetail/14236-CL31A106KBHNNNE/C13585; mpn C3216X5R1H106KT000N -> CL31A106KBHNNNE
- C103, C104, C105, C106: LCSC# C106222 -> C21122; Manufacture YAGEO -> Samsung Electro-Mechanics; SupplLink https://jlcpcb.com/partdetail/Yageo-CC0603KRX7R9BB223/C1062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 -> https://jlcpcb.com/partdetail/21834-CL10B223KB8NNNC/C21122; mpn CC0603KRX7R9BB223 -> CL10B223KB8NNNC
- C107, C110: LCSC# C5162354 -> C249985; Manufacture ROQANG -> Lelon; SupplLink https://jlcpcb.com/partdetail/Roqang-CS1H331MCRG10/C5162354 -> https://jlcpcb.com/partdetail/Lelon-VZT331M1HTR1010/C249985; mpn CS1H331M-CRG10 -> VZT331M1HTR-1010
- C109, C112, C117, C118: LCSC# C1591 -> C14663; Manufacture Samsung Electro-Mechanics -> YAGEO; SupplLink https://jlcpcb.com/partdetail/1943-CL10B104KB8NNNC/C1591 -> https://jlcpcb.com/partdetail/Yageo-CC0603KRX7R9BB104/C14663; mpn CL10B104KB8NNNC -> CC0603KRX7R9BB104
- R101, R103, R104, R105: LCSC# C319934 -> C25744; Manufacture Viking Tech -> UNI-ROYAL(Uniroyal Elec); SupplLink https://jlcpcb.com/partdetail/VikingTech-AR02DTC1002/C319934 -> https://jlcpcb.com/partdetail/26487-0402WGF1002TCE/C25744; mpn AR02DTC1002 -> 0402WGF1002TCE
- R102: value 1R1 -> 1; LCSC# C168518 -> C17928; Manufacture Walsin Tech Corp -> UNI-ROYAL(Uniroyal Elec); SupplLink https://jlcpcb.com/partdetail/Walsin_TechCorp-WR12W1R10FTL/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 -> https://jlcpcb.com/partdetail/18616-1206W4F100KT5E/C17928; mpn WR12W1R10FTL -> 1206W4F100KT5E
- R106, R107: mpn 0402WGF2001TCE -> 0402WGF2001TCE
- U105, U106: mpn ACS712ELCTR-20A-T -> ACS712ELCTR-20A-T

Commit message: Add filter capacitors
Signed-off-by: Benedikt Spranger <b.spranger@linutronix.de>
Parts:
- added C119, C120: 100n, Capacitor_SMD:C_0603_1608Metric, symbol Device:C
Connections:
- net +5V: now also C119.1, C120.1
- net GND: now also C119.2, C120.2
